File: UV_Enclosure_Complete/UV_Enclosure_Complete.kicad_pcb (KiCad board)
At the start: 2 copper layers, 53 parts, among them J1 Spare I/O Header, J2 USB Header, J3 5V Header, J4 Top Panel 1, J5 Top Panel 2, J6 Bottom Panel 1, J7 Bottom Panel 2, J8 Barrel_Jack, P1 Serial header, P2 Programming_Header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

Commit message: Added pull up resistor on V_PP and started routing traces.
Parts:
- added R21: 10kR, Resistors_THT:R_Axial_DIN0309_L9.0mm_D3.2mm_P12.70mm_Horizontal, F.Cu at (132.1, 62.2)
- R1: value R -> 100kR
- R2: value R -> 10kR
- R3: value R -> 1kR
Routing:
- net +12V: track 0.00 -> 285.7 mm
- net GND: track 0.00 -> 156.5 mm
- net +5V: track 0.00 -> 97.9 mm
- net Net-(R6-Pad1): track 0.00 -> 22.2 mm
- net Net-(R5-Pad1): track 0.00 -> 22.2 mm
- net Net-(R4-Pad1): track 0.00 -> 22.2 mm
- net Net-(R12-Pad1): track 0.00 -> 22.2 mm
- net Net-(F1-Pad2): track 0.00 -> 11.4 mm
- net V_PP: track 0.00 -> 6.88 mm
- net Net-(D9-Pad1): track 0.00 -> 6.66 mm
- net Net-(D3-Pad1): track 0.00 -> 5.08 mm
- net Net-(D8-Pad1): track 0.00 -> 5.08 mm
- net Net-(D5-Pad1): track 0.00 -> 5.08 mm
- net Net-(D4-Pad1): track 0.00 -> 5.08 mm
